Commit message: 尝试加入模型

File: mani_skill/assets/robots/panda/panda_v2_back_up.urdf (robot description, URDF)
Before this commit: robot panda, 15 links, 14 joints
Links:
- removed link base_frame
- removed link gripper_frame
- removed link part_1
- removed link part_3
- removed link part_4
- removed link spur_gear__25_teeth
- added link panda_hand, mass 0.73; collision mesh filename=franka_description/meshes/collision/hand.stl; visual mesh filename=franka_description/meshes/visual/hand.glb
- added link panda_hand_tcp
- added link panda_leftfinger, mass 0.015; collision box size=17.5e-3 15.2e-3 18.5e-3; collision box size=17.5e-3 7e-3 23.5e-3
- added link panda_leftfinger_pad
- added link panda_rightfinger, mass 0.015; collision box size=17.5e-3 15.2e-3 18.5e-3; collision box size=17.5e-3 7e-3 23.5e-3
- added link panda_rightfinger_pad
Joints:
- removed joint base_frame_frame
- removed joint gripper_frame_frame
- removed joint gripper_lerft
- removed joint gripper_mount
- removed joint gripper_right
- removed joint motor_gear
- added joint panda_finger_joint1: type prismatic, parent panda_hand, child panda_leftfinger, origin xyz=0 0 0.0584 rpy=0 0 0, axis 0 1 0, limit lower=0.0 upper=0.04 effort=100 velocity=0.2
- added joint panda_finger_joint2: type prismatic, parent panda_hand, child panda_rightfinger, origin xyz=0 0 0.0584 rpy=0 0 0, axis 0 -1 0, limit lower=0.0 upper=0.04 effort=100 velocity=0.2, mimic joint=panda_finger_joint1
- added joint panda_hand_joint: type fixed, parent panda_link8, child panda_hand, origin xyz=0 0 0 rpy=0 0 -0.7853981633974483
- added joint panda_hand_tcp_joint: type fixed, parent panda_hand, child panda_hand_tcp, origin xyz=0 0 0.1034 rpy=0 0 0
- added joint panda_leftfinger_pad_joint: type fixed, parent panda_leftfinger, child panda_leftfinger_pad, origin xyz=0 0 0.0455 rpy=0 0 0
- added joint panda_rightfinger_pad_joint: type fixed, parent panda_rightfinger, child panda_rightfinger_pad, origin xyz=0 0 0.0455 rpy=0 0 0
