Commit message: t

File: mani_skill/assets/robots/panda/panda_v2_2.urdf (robot description, URDF)
Before this commit: robot panda, 16 links, 15 joints
Links:
- removed link part_3
- added link panda_hand_1, mass 1e-9
- link panda_hand: mass 1e-9 -> 0.0837641; geometry collision mesh filename=gripper/convex_decomposition/part_3_parts_00000.stl; collision mesh filename=gripper/convex_decomposition/part_3_parts_00001.stl
Joints:
- removed joint panda_hand_frame
- added joint panda_hand_1_frame: type fixed, parent panda_hand, child panda_hand_1, origin xyz=1.47451e-17 2.91244e-18 0 rpy=-1.22465e-16 6.12323e-17 -4.59169e-49, axis 0 0 0
- joint panda_finger_joint1: parent part_3 -> panda_hand
- joint panda_finger_joint2: parent part_3 -> panda_hand
- joint panda_hand_joint: child part_3 -> panda_hand; origin xyz=0 0 0.001 rpy=0 0 0 -> xyz=0 0 0 rpy=0 0 0
- joint panda_hand_tcp_frame: parent part_3 -> panda_hand
