Commit message: 尝试加入模型

File: mani_skill/assets/robots/panda/panda_v2.urdf (robot description, URDF)
Before this commit: robot panda, 15 links, 14 joints
Links:
- removed link gripper_frame
- added link panda_hand_tcp, mass 1e-9
- link part_1: geometry collision mesh filename=gripper/part_1.stl; collision mesh filename=gripper/part_2.stl
- link part_3: geometry collision mesh filename=gripper/main.stl; collision mesh filename=gripper/part_12.stl
- link part_4: geometry collision mesh filename=gripper/part_4.stl; collision mesh filename=gripper/part_5.stl
- link spur_gear__25_teeth: geometry collision mesh filename=gripper/ac1.stl; collision mesh filename=gripper/spur_gear__25_teeth.stl
Joints:
- joint gripper_frame_frame: child gripper_frame -> panda_hand_tcp

Commit message: 尝试加入模型

File: mani_skill/assets/robots/panda/panda_v2.urdf (robot description, URDF)
Before this commit: robot panda, 15 links, 14 joints
Joints:
- removed joint gripper_lerft
- removed joint gripper_right
- added joint panda_finger_joint1: type revolute, parent part_3, child part_4, origin xyz=-0.10918 0.0134056 0.015 rpy=3.09945e-39 -7.84907e-40 1.74533e-06, axis 0 0 1, limit lower=-1.21337e-18 upper=0.69813 effort=10 velocity=10
- added joint panda_finger_joint2: type revolute, parent part_3, child part_1, origin xyz=-0.10918 -0.0134056 0.015 rpy=-5.76407e-17 -9.46633e-16 -1.74533e-06, axis 0 0 1, limit lower=-0.69813 upper=1.91986e-06 effort=10 velocity=10, mimic joint=panda_finger_joint1 multiplier=-1.0
- joint motor_gear: mimic joint=gripper_right multiplier=-0.8 -> joint=panda_finger_joint2 multiplier=-0.8

Commit message: 尝试加入模型

File: mani_skill/assets/robots/panda/panda_v2.urdf (robot description, URDF)
Before this commit: robot panda, 15 links, 14 joints
Links:
- removed link part_3
- added link panda_hand, mass 1e-09; collision mesh filename=gripper/main.stl; collision mesh filename=gripper/part_12.stl
Joints:
- joint base_frame_frame: parent part_3 -> panda_hand
- joint gripper_mount: child part_3 -> panda_hand
- joint motor_gear: parent part_3 -> panda_hand
- joint panda_finger_joint1: parent part_3 -> panda_hand
- joint panda_finger_joint2: parent part_3 -> panda_hand

Commit message: 尝试加入模型

File: mani_skill/assets/robots/panda/panda_v2.urdf (robot description, URDF)
Before this commit: robot panda, 15 links, 14 joints
Links:
- removed link part_1
- removed link part_4
- added link panda_leftfinger, mass 1e-09; collision mesh filename=gripper/part_4.stl; collision mesh filename=gripper/part_5.stl
- added link panda_rightfinger, mass 1e-09; collision mesh filename=gripper/part_1.stl; collision mesh filename=gripper/part_2.stl
Joints:
- joint gripper_frame_frame: parent part_4 -> panda_leftfinger
- joint motor_gear: mimic joint=panda_finger_joint2 multiplier=-0.8 -> joint=panda_finger_joint1 multiplier=-0.8
- joint panda_finger_joint1: child part_4 -> panda_rightfinger; limit lower=-1.21337e-18 upper=0.69813 effort=10 velocity=10 -> lower=-0.69813 upper=1.91986e-06 effort=10 velocity=10; mimic (none) -> joint=panda_finger_joint2 multiplier=-1.0; origin xyz=-0.10918 0.0134056 0.015 rpy=3.09945e-39 -7.84907e-40 1.74533e-06 -> xyz=-0.10918 -0.0134056 0.015 rpy=-5.76407e-17 -9.46633e-16 -1.74533e-06
- joint panda_finger_joint2: child part_1 -> panda_leftfinger; limit lower=-0.69813 upper=1.91986e-06 effort=10 velocity=10 -> lower=-1.21337e-18 upper=0.69813 effort=10 velocity=10; mimic joint=panda_finger_joint1 multiplier=-1.0 -> (none); origin xyz=-0.10918 -0.0134056 0.015 rpy=-5.76407e-17 -9.46633e-16 -1.74533e-06 -> xyz=-0.10918 0.0134056 0.015 rpy=3.09945e-39 -7.84907e-40 1.74533e-06

Commit message: 尝试加入模型

File: mani_skill/assets/robots/panda/panda_v2.urdf (robot description, URDF)
Before this commit: robot panda, 15 links, 14 joints
Links:
- removed link spur_gear__25_teeth
Joints:
- removed joint motor_gear

Commit message: 尝试加入模型

File: mani_skill/assets/robots/panda/panda_v2.urdf (robot description, URDF)
Before this commit: robot panda, 14 links, 13 joints
Links:
- removed link base_frame
- added link panda_rightfinger_pad, mass 1e-9
- link panda_hand: mass 1e-09 -> 1e-9; geometry 
- link panda_leftfinger: mass 1e-09 -> 0.0322882; geometry collision mesh filename=gripper/panda_leftfinger_collision.stl; visual mesh filename=gripper/panda_leftfinger_visual.stl
- link panda_rightfinger: mass 1e-09 -> 0.0320815; geometry collision mesh filename=gripper/panda_rightfinger_collision.stl; visual mesh filename=gripper/panda_rightfinger_visual.stl
Joints:
- removed joint base_frame_frame
- removed joint gripper_frame_frame
- removed joint panda_finger_joint1
- removed joint panda_finger_joint2
- added joint finger_joint1: type revolute, parent panda_hand, child panda_leftfinger, origin xyz=-0.10918 0.0134056 0.015 rpy=2.18003e-16 -8.41922e-16 1.74533e-09, axis 0 0 1, limit lower=0 upper=0.698132 effort=10 velocity=10, mimic joint=finger_joint2 multiplier=-1.0
- added joint finger_joint2: type revolute, parent panda_hand, child panda_rightfinger, origin xyz=-0.10918 -0.0134056 0.015 rpy=-2.98866e-24 2.19338e-30 -1.74533e-09, axis 0 0 1, limit lower=-0.698132 upper=1.91986e-08 effort=10 velocity=10
- added joint panda_hand_frame: type fixed, parent panda_hand, child panda_hand, origin xyz=-0.160364 -1.73472e-18 0.00598 rpy=1.5708 -0 1.5708, axis 0 0 0
- added joint panda_hand_tcp_frame: type fixed, parent panda_leftfinger, child panda_hand_tcp, origin xyz=0.058726 0.015782 0.005 rpy=5.41441e-17 1.22433e-17 -0.222385, axis 0 0 0
- added joint panda_rightfinger_pad_frame: type fixed, parent panda_rightfinger, child panda_rightfinger_pad, origin xyz=0.058726 -0.015782 0.005 rpy=-5.41441e-17 1.22433e-17 0.222385, axis 0 0 0

Commit message: 尝试加入模型

File: mani_skill/assets/robots/panda/panda_v2.urdf (robot description, URDF)
Before this commit: robot panda, 14 links, 14 joints
Links:
- added link part_3, mass 0.0837641; collision mesh filename=package://assets/merged/part_3_collision.stl; visual mesh filename=package://assets/merged/part_3_visual.stl
- link panda_leftfinger: geometry collision mesh filename=package://assets/merged/panda_leftfinger_collision.stl; visual mesh filename=package://assets/merged/panda_leftfinger_visual.stl
- link panda_rightfinger: geometry collision mesh filename=package://assets/merged/panda_rightfinger_collision.stl; visual mesh filename=package://assets/merged/panda_rightfinger_visual.stl
Joints:
- removed joint gripper_mount
- added joint panda_hand_joint: type fixed, parent panda_link8, child panda_hand, origin xyz=0 0 0 rpy=0 0 0
- joint finger_joint1: parent panda_hand -> part_3
- joint finger_joint2: parent panda_hand -> part_3
- joint panda_hand_frame: parent panda_hand -> part_3

Commit message: 尝试加入模型

File: mani_skill/assets/robots/panda/panda_v2.urdf (robot description, URDF)
Before this commit: robot panda, 15 links, 14 joints
Links:
- added link panda_leftfinger_pad, mass 1e-9
Joints:
- added joint panda_leftfinger_pad_frame: type fixed, parent panda_leftfinger, child panda_leftfinger_pad, origin xyz=0.058726 0.015782 0.005 rpy=5.41441e-17 1.22433e-17 -0.222385, axis 0 0 0
- joint panda_hand_tcp_frame: origin xyz=0.058726 0.015782 0.005 rpy=5.41441e-17 1.22433e-17 -0.222385 -> xyz=0.0074957 -1.73472e-18 0.00598 rpy=0 -6.12323e-17 0; parent panda_leftfinger -> part_3

Commit message: 尝试加入模型

File: mani_skill/assets/robots/panda/panda_v2.urdf (robot description, URDF)
Before this commit: robot panda, 16 links, 15 joints
Links:
- link panda_leftfinger: geometry collision mesh filename=gripper/panda_leftfinger_collision.stl; visual mesh filename=gripper/panda_leftfinger_visual.stl
- link panda_rightfinger: geometry collision mesh filename=gripper/panda_rightfinger_collision.stl; visual mesh filename=gripper/panda_rightfinger_visual.stl
- link part_3: geometry collision mesh filename=gripper/part_3_collision.stl; visual mesh filename=gripper/part_3_visual.stl
Joints:
- joint panda_hand_joint: child panda_hand -> part_3

Commit message: 尝试加入模型

File: mani_skill/assets/robots/panda/panda_v2.urdf (robot description, URDF)
Before this commit: robot panda, 16 links, 15 joints
Links:
- link panda_leftfinger: geometry collision mesh filename=gripper/convex_decomposition/panda_leftfinger_parts_00000.s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; collision mesh filename=gripper/convex_decomposition/panda_leftfinger_parts_00001.s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
- link panda_rightfinger: geometry collision mesh filename=gripper/convex_decomposition/panda_rightfinger_parts_00000.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; collision mesh filename=gripper/convex_decomposition/panda_rightfinger_parts_00001.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
- link part_3: geometry collision mesh filename=gripper/convex_decomposition/part_3_parts_00000.stl; collision mesh filename=gripper/convex_decomposition/part_3_parts_00001.stl
Joints:
- removed joint finger_joint1
- removed joint finger_joint2
- added joint panda_finger_joint1: type revolute, parent part_3, child panda_leftfinger, origin xyz=-0.10918 0.0134056 0.015 rpy=2.18003e-16 -8.41922e-16 1.74533e-09, axis 0 0 1, limit lower=0 upper=0.698132 effort=10 velocity=10, mimic joint=panda_finger_joint2 multiplier=-1.0
- added joint panda_finger_joint2: type revolute, parent part_3, child panda_rightfinger, origin xyz=-0.10918 -0.0134056 0.015 rpy=-2.98866e-24 2.19338e-30 -1.74533e-09, axis 0 0 1, limit lower=-0.698132 upper=1.91986e-08 effort=10 velocity=10

Commit message: ok

File: mani_skill/assets/robots/panda/panda_v2.urdf (robot description, URDF)
Before this commit: robot panda, 16 links, 15 joints
Joints:
- joint panda_hand_joint: origin xyz=0 0 0 rpy=0 0 0 -> xyz=0 0 0.16 rpy=0 -1.5708 2.38562

Commit message: 尝试加入模型

File: mani_skill/assets/robots/panda/panda_v2.urdf (robot description, URDF)
Before this commit: robot panda, 16 links, 15 joints
Links:
- removed link part_3
- link panda_hand: mass 1e-9 -> 0.73; geometry collision mesh filename=franka_description/meshes/collision/hand.stl; visual mesh filename=franka_description/meshes/visual/hand.glb
- link panda_hand_tcp: mass 1e-9 -> None
- link panda_leftfinger: mass 0.0322882 -> 0.015; geometry collision box size=17.5e-3 15.2e-3 18.5e-3; collision box size=17.5e-3 7e-3 23.5e-3
- link panda_leftfinger_pad: mass 1e-9 -> None
- link panda_rightfinger: mass 0.0320815 -> 0.015; geometry collision box size=17.5e-3 15.2e-3 18.5e-3; collision box size=17.5e-3 7e-3 23.5e-3
- link panda_rightfinger_pad: mass 1e-9 -> None
Joints:
- removed joint panda_hand_frame
- removed joint panda_hand_tcp_frame
- removed joint panda_leftfinger_pad_frame
- removed joint panda_rightfinger_pad_frame
- added joint panda_hand_tcp_joint: type fixed, parent panda_hand, child panda_hand_tcp, origin xyz=0 0 0.1034 rpy=0 0 0
- added joint panda_leftfinger_pad_joint: type fixed, parent panda_leftfinger, child panda_leftfinger_pad, origin xyz=0 0 0.0455 rpy=0 0 0
- added joint panda_rightfinger_pad_joint: type fixed, parent panda_rightfinger, child panda_rightfinger_pad, origin xyz=0 0 0.0455 rpy=0 0 0
- joint panda_finger_joint1: axis 0 0 1 -> 0 1 0; limit lower=0 upper=0.698132 effort=10 velocity=10 -> lower=0.0 upper=0.04 effort=100 velocity=0.2; mimic joint=panda_finger_joint2 multiplier=-1.0 -> (none); origin xyz=-0.10918 0.0134056 0.015 rpy=2.18003e-16 -8.41922e-16 1.74533e-09 -> xyz=0 0 0.0584 rpy=0 0 0; parent part_3 -> panda_hand; type revolute -> prismatic
- joint panda_finger_joint2: axis 0 0 1 -> 0 -1 0; limit lower=-0.698132 upper=1.91986e-08 effort=10 velocity=10 -> lower=0.0 upper=0.04 effort=100 velocity=0.2; mimic (none) -> joint=panda_finger_joint1; origin xyz=-0.10918 -0.0134056 0.015 rpy=-2.98866e-24 2.19338e-30 -1.74533e-09 -> xyz=0 0 0.0584 rpy=0 0 0; parent part_3 -> panda_hand; type revolute -> prismatic
- joint panda_hand_joint: child part_3 -> panda_hand; origin xyz=0 0 0.16 rpy=0 -1.5708 2.38562 -> xyz=0 0 0 rpy=0 0 -0.7853981633974483

Commit message: 尝试加入模型

File: mani_skill/assets/robots/panda/panda_v2.urdf (robot description, URDF)
Before this commit: robot panda, 15 links, 14 joints
Links:
- added link part_3, mass 0.0837641; collision mesh filename=gripper/convex_decomposition/part_3_parts_00000.stl; collision mesh filename=gripper/convex_decomposition/part_3_parts_00001.stl
- link panda_hand: mass 0.73 -> 1e-9; geometry 
- link panda_hand_tcp: mass None -> 1e-9
- link panda_leftfinger: mass 0.015 -> 0.0322882; geometry collision mesh filename=gripper/convex_decomposition/panda_leftfinger_parts_00000.s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; collision mesh filename=gripper/convex_decomposition/panda_leftfinger_parts_00001.s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
- link panda_leftfinger_pad: mass None -> 1e-9
- link panda_rightfinger: mass 0.015 -> 0.0320815; geometry collision mesh filename=gripper/convex_decomposition/panda_rightfinger_parts_00000.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; collision mesh filename=gripper/convex_decomposition/panda_rightfinger_parts_00001.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
- link panda_rightfinger_pad: mass None -> 1e-9
Joints:
- removed joint panda_hand_tcp_joint
- removed joint panda_leftfinger_pad_joint
- removed joint panda_rightfinger_pad_joint
- added joint panda_hand_frame: type fixed, parent part_3, child panda_hand, origin xyz=-0.160364 -1.73472e-18 0.00598 rpy=1.5708 -0 1.5708, axis 0 0 0
- added joint panda_hand_tcp_frame: type fixed, parent part_3, child panda_hand_tcp, origin xyz=0.0074957 -1.73472e-18 0.00598 rpy=0 -6.12323e-17 0, axis 0 0 0
- added joint panda_leftfinger_pad_frame: type fixed, parent panda_leftfinger, child panda_leftfinger_pad, origin xyz=0.058726 0.015782 0.005 rpy=5.41441e-17 1.22433e-17 -0.222385, axis 0 0 0
- added joint panda_rightfinger_pad_frame: type fixed, parent panda_rightfinger, child panda_rightfinger_pad, origin xyz=0.058726 -0.015782 0.005 rpy=-5.41441e-17 1.22433e-17 0.222385, axis 0 0 0
- joint panda_finger_joint1: axis 0 1 0 -> 0 0 1; limit lower=0.0 upper=0.04 effort=100 velocity=0.2 -> lower=0 upper=0.698132 effort=10 velocity=10; mimic (none) -> joint=panda_finger_joint2 multiplier=-1.0; origin xyz=0 0 0.0584 rpy=0 0 0 -> xyz=-0.10918 0.0134056 0.015 rpy=2.18003e-16 -8.41922e-16 1.74533e-09; parent panda_hand -> part_3; type prismatic -> revolute
- joint panda_finger_joint2: axis 0 -1 0 -> 0 0 1; limit lower=0.0 upper=0.04 effort=100 velocity=0.2 -> lower=-0.698132 upper=1.91986e-08 effort=10 velocity=10; mimic joint=panda_finger_joint1 -> (none); origin xyz=0 0 0.0584 rpy=0 0 0 -> xyz=-0.10918 -0.0134056 0.015 rpy=-2.98866e-24 2.19338e-30 -1.74533e-09; parent panda_hand -> part_3; type prismatic -> revolute
- joint panda_hand_joint: child panda_hand -> part_3; origin xyz=0 0 0 rpy=0 0 -0.7853981633974483 -> xyz=0 0 0.16 rpy=0 -1.5708 2.38562

Commit message: 尝试加入模型

File: mani_skill/assets/robots/panda/panda_v2.urdf (robot description, URDF)
Before this commit: robot panda, 16 links, 15 joints
Joints:
- joint panda_leftfinger_pad_frame: origin xyz=0.058726 0.015782 0.005 rpy=5.41441e-17 1.22433e-17 -0.222385 -> xyz=0.11668 -0.0134056 -0.009 rpy=6.12323e-17 7.88861e-31 -3.46945e-16
- joint panda_rightfinger_pad_frame: origin xyz=0.058726 -0.015782 0.005 rpy=-5.41441e-17 1.22433e-17 0.222385 -> xyz=0.11668 0.0134056 -0.009 rpy=-6.12323e-17 -2.80596e-32 3.46945e-16

Commit message: 尝试加入模型

File: mani_skill/assets/robots/panda/panda_v2.urdf (robot description, URDF)
Before this commit: robot panda, 15 links, 14 joints
Joints:
- joint panda_finger_joint1: limit lower=0.0 upper=0.04 effort=100 velocity=0.2 -> lower=0.0 upper=0.6 effort=100 velocity=0.2
- joint panda_finger_joint2: limit lower=0.0 upper=0.04 effort=100 velocity=0.2 -> lower=0.0 upper=0.6 effort=100 velocity=0.2

Commit message: 尝试加入模型

File: mani_skill/assets/robots/panda/panda_v2.urdf (robot description, URDF)
Before this commit: robot panda, 15 links, 14 joints
Joints:
- joint panda_finger_joint1: limit lower=0.0 upper=0.6 effort=100 velocity=0.2 -> lower=0.0 upper=0.04 effort=100 velocity=0.2
- joint panda_finger_joint2: limit lower=0.0 upper=0.6 effort=100 velocity=0.2 -> lower=0.0 upper=0.04 effort=100 velocity=0.2

File: mani_skill/assets/robots/panda/panda_v21.urdf (robot description, URDF)
Before this commit: robot panda, 16 links, 15 joints
Joints:
- joint panda_finger_joint1: limit lower=0 upper=0.698132 effort=10 velocity=10 -> lower=0 upper=0.698132 effort=10 velocity=0.2
- joint panda_finger_joint2: limit lower=-0.698132 upper=1.91986e-08 effort=10 velocity=10 -> lower=-0.698132 upper=1.91986e-08 effort=10 velocity=0.2

Commit message: 尝试加入模型

File: mani_skill/assets/robots/panda/panda_v2.urdf (robot description, URDF)
Before this commit: robot panda, 15 links, 14 joints
Links:
- added link part_3, mass 0.0837641; collision mesh filename=gripper/convex_decomposition/part_3_parts_00000.stl; collision mesh filename=gripper/convex_decomposition/part_3_parts_00001.stl
- link panda_hand: mass 0.73 -> 1e-9; geometry 
- link panda_hand_tcp: mass None -> 1e-9
- link panda_leftfinger: mass 0.015 -> 0.0322882; geometry collision mesh filename=gripper/convex_decomposition/panda_leftfinger_parts_00000.s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; collision mesh filename=gripper/convex_decomposition/panda_leftfinger_parts_00001.s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
- link panda_leftfinger_pad: mass None -> 1e-9
- link panda_rightfinger: mass 0.015 -> 0.0320815; geometry collision mesh filename=gripper/convex_decomposition/panda_rightfinger_parts_00000.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; collision mesh filename=gripper/convex_decomposition/panda_rightfinger_parts_00001.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
- link panda_rightfinger_pad: mass None -> 1e-9
Joints:
- removed joint panda_hand_tcp_joint
- removed joint panda_leftfinger_pad_joint
- removed joint panda_rightfinger_pad_joint
- added joint panda_hand_frame: type fixed, parent part_3, child panda_hand, origin xyz=-0.160364 -1.73472e-18 0.00598 rpy=1.5708 -0 1.5708, axis 0 0 0
- added joint panda_hand_tcp_frame: type fixed, parent part_3, child panda_hand_tcp, origin xyz=0.0074957 -1.73472e-18 0.00598 rpy=0 -6.12323e-17 0, axis 0 0 0
- added joint panda_leftfinger_pad_frame: type fixed, parent panda_leftfinger, child panda_leftfinger_pad, origin xyz=0.11668 -0.0134056 -0.009 rpy=6.12323e-17 7.88861e-31 -3.46945e-16, axis 0 0 0
- added joint panda_rightfinger_pad_frame: type fixed, parent panda_rightfinger, child panda_rightfinger_pad, origin xyz=0.11668 0.0134056 -0.009 rpy=-6.12323e-17 -2.80596e-32 3.46945e-16, axis 0 0 0
- joint panda_finger_joint1: axis 0 1 0 -> 0 0 1; limit lower=0.0 upper=0.04 effort=100 velocity=0.2 -> lower=0 upper=0.698132 effort=10 velocity=0.2; mimic (none) -> joint=panda_finger_joint2 multiplier=-1.0; origin xyz=0 0 0.0584 rpy=0 0 0 -> xyz=-0.10918 0.0134056 0.015 rpy=2.18003e-16 -8.41922e-16 1.74533e-09; parent panda_hand -> part_3; type prismatic -> revolute
- joint panda_finger_joint2: axis 0 -1 0 -> 0 0 1; limit lower=0.0 upper=0.04 effort=100 velocity=0.2 -> lower=-0.698132 upper=1.91986e-08 effort=10 velocity=0.2; mimic joint=panda_finger_joint1 -> (none); origin xyz=0 0 0.0584 rpy=0 0 0 -> xyz=-0.10918 -0.0134056 0.015 rpy=-2.98866e-24 2.19338e-30 -1.74533e-09; parent panda_hand -> part_3; type prismatic -> revolute
- joint panda_hand_joint: child panda_hand -> part_3; origin xyz=0 0 0 rpy=0 0 -0.7853981633974483 -> xyz=0 0 0.16 rpy=0 -1.5708 2.38562

Commit message: ok

File: mani_skill/assets/robots/panda/panda_v2.urdf (robot description, URDF)
Before this commit: robot panda, 16 links, 15 joints
Joints:
- joint panda_hand_joint: origin xyz=0 0 0.16 rpy=0 -1.5708 2.38562 -> xyz=0 0 0.162 rpy=0 -1.5708 2.38562

Commit message: 尝试加入模型

File: mani_skill/assets/robots/panda/panda_v2.urdf (robot description, URDF)
Before this commit: robot panda, 16 links, 15 joints
Joints:
- joint panda_finger_joint1: limit lower=0 upper=0.698132 effort=10 velocity=0.2 -> lower=0 upper=0.69 effort=10 velocity=0.2
- joint panda_finger_joint2: limit lower=-0.698132 upper=1.91986e-08 effort=10 velocity=0.2 -> lower=-0.69 upper=0 effort=10 velocity=0.2

Commit message: 尝试加入模型

File: mani_skill/assets/robots/panda/panda_v2.urdf (robot description, URDF)
Before this commit: robot panda, 16 links, 15 joints
Joints:
- joint panda_finger_joint1: origin xyz=-0.10918 0.0134056 0.015 rpy=2.18003e-16 -8.41922e-16 1.74533e-09 -> xyz=-0.10918 0.0134056 0.015 rpy=0 0 0
- joint panda_finger_joint2: origin xyz=-0.10918 -0.0134056 0.015 rpy=-2.98866e-24 2.19338e-30 -1.74533e-09 -> xyz=-0.10918 -0.0134056 0.015 rpy=0 0 0

Commit message: 尝试加入模型

File: mani_skill/assets/robots/panda/panda_v2.urdf (robot description, URDF)
Before this commit: robot panda, 16 links, 15 joints
Joints:
- joint panda_finger_joint1: limit lower=0 upper=0.69 effort=10 velocity=0.2 -> lower=0 upper=0.69 effort=10 velocity=0.3; mimic joint=panda_finger_joint2 multiplier=-1.0 -> joint=panda_finger_joint2 multiplier=1.0
- joint panda_finger_joint2: axis 0 0 1 -> 0 0 -1; limit lower=-0.69 upper=0 effort=10 velocity=0.2 -> lower=0.69 upper=0 effort=10 velocity=0.3

Commit message: 尝试加入模型

File: mani_skill/assets/robots/panda/panda_v2.urdf (robot description, URDF)
Before this commit: robot panda, 16 links, 15 joints
Joints:
- joint panda_finger_joint2: limit lower=0.69 upper=0 effort=10 velocity=0.3 -> lower=0 upper=0.69 effort=10 velocity=0.3

Commit message: 尝试加入模型

File: mani_skill/assets/robots/panda/panda_v2.urdf (robot description, URDF)
Before this commit: robot panda, 16 links, 15 joints
Links:
- link panda_leftfinger: geometry collision mesh filename=gripper/convex_decomposition/panda_leftfinger_00000.stl; collision mesh filename=gripper/convex_decomposition/panda_leftfinger_00001.stl
- link panda_rightfinger: geometry collision mesh filename=gripper/convex_decomposition/panda_rightfinger_00000.stl; collision mesh filename=gripper/convex_decomposition/panda_rightfinger_00001.stl
- link part_3: geometry collision mesh filename=gripper/convex_decomposition/main_00000.stl; collision mesh filename=gripper/convex_decomposition/main_00001.stl
Joints:
- joint panda_finger_joint1: limit lower=0 upper=0.69 effort=10 velocity=0.3 -> lower=0 upper=0.69 effort=10 velocity=.3; origin xyz=-0.10918 0.0134056 0.015 rpy=0 0 0 -> xyz=0.00902 -0.0134056 0.0511842 rpy=3.14159 -1.5708 0
- joint panda_finger_joint2: limit lower=0 upper=0.69 effort=10 velocity=0.3 -> lower=0 upper=0.69 effort=10 velocity=10; origin xyz=-0.10918 -0.0134056 0.015 rpy=0 0 0 -> xyz=0.00902 0.0134056 0.0511842 rpy=3.14159 -1.5708 0
- joint panda_hand_frame: origin xyz=-0.160364 -1.73472e-18 0.00598 rpy=1.5708 -0 1.5708 -> xyz=1.47451e-17 2.91244e-18 0 rpy=-1.22465e-16 6.12323e-17 -4.59169e-49
- joint panda_hand_tcp_frame: origin xyz=0.0074957 -1.73472e-18 0.00598 rpy=0 -6.12323e-17 0 -> xyz=2.51535e-17 2.34694e-17 0.16786 rpy=3.14159 -1.5708 0
- joint panda_leftfinger_pad_frame: origin xyz=0.11668 -0.0134056 -0.009 rpy=6.12323e-17 7.88861e-31 -3.46945e-16 -> xyz=0.11668 -0.0134056 -0.009 rpy=6.12323e-17 -2.80378e-32 -3.46945e-16
- joint panda_rightfinger_pad_frame: origin xyz=0.11668 0.0134056 -0.009 rpy=-6.12323e-17 -2.80596e-32 3.46945e-16 -> xyz=0.11668 0.0134056 -0.009 rpy=-6.12323e-17 -7.24343e-32 3.46945e-16
