Commit message: 尝试加入模型

File: mani_skill/assets/robots/panda/panda_v2.urdf (robot description, URDF)
Before this commit: robot panda, 16 links, 15 joints
Links:
- link panda_leftfinger: geometry collision mesh filename=gripper/convex_decomposition/panda_leftfinger_parts_00000.s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; collision mesh filename=gripper/convex_decomposition/panda_leftfinger_parts_00001.s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
- link panda_rightfinger: geometry collision mesh filename=gripper/convex_decomposition/panda_rightfinger_parts_00000.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; collision mesh filename=gripper/convex_decomposition/panda_rightfinger_parts_00001.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
- link part_3: geometry collision mesh filename=gripper/convex_decomposition/part_3_parts_00000.stl; collision mesh filename=gripper/convex_decomposition/part_3_parts_00001.stl
Joints:
- joint panda_finger_joint1: limit lower=0 upper=0.69 effort=10 velocity=.3 -> lower=0 upper=0.69 effort=10 velocity=0.3
- joint panda_finger_joint2: limit lower=0 upper=0.69 effort=10 velocity=10 -> lower=0.0 upper=0.69 effort=10 velocity=0.3

Commit message: 尝试加入模型

File: mani_skill/assets/robots/panda/panda_v2.urdf (robot description, URDF)
Before this commit: robot panda, 16 links, 15 joints
Joints:
- joint panda_hand_joint: origin xyz=0 0 0.162 rpy=0 -1.5708 2.38562 -> xyz=0 0 0 rpy=0 0 0

Commit message: 尝试加入模型

File: mani_skill/assets/robots/panda/panda_v2.urdf (robot description, URDF)
Before this commit: robot panda, 16 links, 15 joints
Joints:
- joint panda_hand_joint: origin xyz=0 0 0 rpy=0 0 0 -> xyz=0 0 0.01 rpy=0 0 0

Commit message: 尝试加入模型

File: mani_skill/assets/robots/panda/panda_v2.urdf (robot description, URDF)
Before this commit: robot panda, 16 links, 15 joints
Joints:
- joint panda_hand_joint: origin xyz=0 0 0.01 rpy=0 0 0 -> xyz=0 0 0.0001 rpy=0 0 0

Commit message: 尝试加入模型

File: mani_skill/assets/robots/panda/panda_v2.urdf (robot description, URDF)
Before this commit: robot panda, 16 links, 15 joints
Joints:
- joint panda_hand_joint: origin xyz=0 0 0.0001 rpy=0 0 0 -> xyz=0 0 0.001 rpy=0 0 0

Commit message: 尝试加入模型

File: mani_skill/assets/robots/panda/panda_v2.urdf (robot description, URDF)
Before this commit: robot panda, 16 links, 15 joints
Joints:
- joint panda_hand_tcp_frame: origin xyz=2.51535e-17 2.34694e-17 0.16786 rpy=3.14159 -1.5708 0 -> xyz=2.51535e-17 2.34694e-17 0.16786 rpy=-1.22465e-16 6.12323e-17 -4.59169e-49

Commit message: 尝试加入模型

File: mani_skill/assets/robots/panda/panda_v2.urdf (robot description, URDF)
Before this commit: robot panda, 16 links, 15 joints
Joints:
- joint panda_finger_joint1: limit lower=0 upper=0.69 effort=10 velocity=0.3 -> lower=-0.184007 upper=0.514125 effort=10 velocity=0.3; origin xyz=0.00902 -0.0134056 0.0511842 rpy=3.14159 -1.5708 0 -> xyz=0.00902 -0.0134056 0.0511842 rpy=-1.5708 -1.38679 -1.5708
- joint panda_finger_joint2: limit lower=0.0 upper=0.69 effort=10 velocity=0.3 -> lower=0.184007 upper=-0.514125 effort=10 velocity=0.3; origin xyz=0.00902 0.0134056 0.0511842 rpy=3.14159 -1.5708 0 -> xyz=0.00902 0.0134056 0.0511842 rpy=1.5708 -1.38679 1.5708
- joint panda_leftfinger_pad_frame: origin xyz=0.11668 -0.0134056 -0.009 rpy=6.12323e-17 -2.80378e-32 -3.46945e-16 -> xyz=0.11668 -0.0134056 -0.009 rpy=3.14159 -1.5708 0
- joint panda_rightfinger_pad_frame: origin xyz=0.11668 0.0134056 -0.009 rpy=-6.12323e-17 -7.24343e-32 3.46945e-16 -> xyz=0.11668 0.0134056 -0.009 rpy=-3.14159 -1.5708 0

Commit message: 尝试加入模型

File: mani_skill/assets/robots/panda/panda_v2.urdf (robot description, URDF)
Before this commit: robot panda, 16 links, 15 joints
Joints:
- joint panda_finger_joint2: limit lower=0.184007 upper=-0.514125 effort=10 velocity=0.3 -> lower=-0.184007 upper=0.514125 effort=10 velocity=0.3

Commit message: 尝试加入模型

File: mani_skill/assets/robots/panda/panda_v2.urdf (robot description, URDF)
Before this commit: robot panda, 16 links, 15 joints
Joints:
- joint panda_finger_joint1: limit lower=-0.184007 upper=0.514125 effort=10 velocity=0.3 -> lower=-0.185 upper=0.5 effort=10 velocity=0.3
- joint panda_finger_joint2: limit lower=-0.184007 upper=0.514125 effort=10 velocity=0.3 -> lower=-0.185 upper=0.5 effort=10 velocity=0.3

Commit message: 尝试加入模型

File: mani_skill/assets/robots/panda/panda_v2.urdf (robot description, URDF)
Before this commit: robot panda, 16 links, 15 joints
Joints:
- joint panda_finger_joint1: limit lower=-0.185 upper=0.5 effort=10 velocity=0.3 -> lower=-0.185 upper=0.5 effort=100 velocity=10
- joint panda_finger_joint2: limit lower=-0.185 upper=0.5 effort=10 velocity=0.3 -> lower=-0.185 upper=0.5 effort=100 velocity=10

Commit message: 尝试加入模型

File: mani_skill/assets/robots/panda/panda_v2.urdf (robot description, URDF)
Before this commit: robot panda, 16 links, 15 joints
Joints:
- joint panda_finger_joint2: limit lower=-0.185 upper=0.5 effort=100 velocity=10 -> lower=-0.185 upper=0.5 effort=100 velocity=100

Commit message: 尝试加入模型

File: mani_skill/assets/robots/panda/panda_v2.urdf (robot description, URDF)
Before this commit: robot panda, 16 links, 15 joints
Joints:
- joint panda_finger_joint2: limit lower=-0.185 upper=0.5 effort=100 velocity=100 -> lower=-0.185 upper=0.5 effort=100 velocity=10

Commit message: 尝试加入模型

File: mani_skill/assets/robots/panda/panda_v2.urdf (robot description, URDF)
Before this commit: robot panda, 16 links, 15 joints
Links:
- removed link part_3
- link panda_hand: mass 1e-9 -> 0.73; geometry collision mesh filename=franka_description/meshes/collision/hand.stl; visual mesh filename=franka_description/meshes/visual/hand.glb
- link panda_hand_tcp: mass 1e-9 -> None
- link panda_leftfinger: mass 0.0322882 -> 0.015; geometry collision box size=17.5e-3 15.2e-3 18.5e-3; collision box size=17.5e-3 7e-3 23.5e-3
- link panda_leftfinger_pad: mass 1e-9 -> None
- link panda_rightfinger: mass 0.0320815 -> 0.015; geometry collision box size=17.5e-3 15.2e-3 18.5e-3; collision box size=17.5e-3 7e-3 23.5e-3
- link panda_rightfinger_pad: mass 1e-9 -> None
Joints:
- removed joint panda_hand_frame
- removed joint panda_hand_tcp_frame
- removed joint panda_leftfinger_pad_frame
- removed joint panda_rightfinger_pad_frame
- added joint panda_hand_tcp_joint: type fixed, parent panda_hand, child panda_hand_tcp, origin xyz=0 0 0.1034 rpy=0 0 0
- added joint panda_leftfinger_pad_joint: type fixed, parent panda_leftfinger, child panda_leftfinger_pad, origin xyz=0 0 0.0455 rpy=0 0 0
- added joint panda_rightfinger_pad_joint: type fixed, parent panda_rightfinger, child panda_rightfinger_pad, origin xyz=0 0 0.0455 rpy=0 0 0
- joint panda_finger_joint1: axis 0 0 1 -> 0 1 0; limit lower=-0.185 upper=0.5 effort=100 velocity=10 -> lower=0.0 upper=0.04 effort=100 velocity=0.2; mimic joint=panda_finger_joint2 multiplier=1.0 -> (none); origin xyz=0.00902 -0.0134056 0.0511842 rpy=-1.5708 -1.38679 -1.5708 -> xyz=0 0 0.0584 rpy=0 0 0; parent part_3 -> panda_hand; type revolute -> prismatic
- joint panda_finger_joint2: axis 0 0 -1 -> 0 -1 0; limit lower=-0.185 upper=0.5 effort=100 velocity=10 -> lower=0.0 upper=0.04 effort=100 velocity=0.2; mimic (none) -> joint=panda_finger_joint1; origin xyz=0.00902 0.0134056 0.0511842 rpy=1.5708 -1.38679 1.5708 -> xyz=0 0 0.0584 rpy=0 0 0; parent part_3 -> panda_hand; type revolute -> prismatic
- joint panda_hand_joint: child part_3 -> panda_hand; origin xyz=0 0 0.001 rpy=0 0 0 -> xyz=0 0 0 rpy=0 0 -0.7853981633974483

Commit message: t

File: mani_skill/assets/robots/panda/panda_v2.urdf (robot description, URDF)
Before this commit: robot panda, 15 links, 14 joints
Links:
- added link panda_hand_1, mass 1e-9
- link panda_hand: mass 0.73 -> 0.0837641; geometry collision mesh filename=gripper/convex_decomposition/part_3_parts_00000.stl; collision mesh filename=gripper/convex_decomposition/part_3_parts_00001.stl
- link panda_hand_tcp: mass None -> 1e-9
- link panda_leftfinger: mass 0.015 -> 0.0322882; geometry collision mesh filename=gripper/convex_decomposition/panda_leftfinger_parts_00000.s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; collision mesh filename=gripper/convex_decomposition/panda_leftfinger_parts_00001.s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
- link panda_leftfinger_pad: mass None -> 1e-9
- link panda_rightfinger: mass 0.015 -> 0.0320815; geometry collision mesh filename=gripper/convex_decomposition/panda_rightfinger_parts_00000.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; collision mesh filename=gripper/convex_decomposition/panda_rightfinger_parts_00001.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
- link panda_rightfinger_pad: mass None -> 1e-9
Joints:
- removed joint panda_hand_tcp_joint
- removed joint panda_leftfinger_pad_joint
- removed joint panda_rightfinger_pad_joint
- added joint panda_hand_1_frame: type fixed, parent panda_hand, child panda_hand_1, origin xyz=1.47451e-17 2.91244e-18 0 rpy=-1.22465e-16 6.12323e-17 -4.59169e-49, axis 0 0 0
- added joint panda_hand_tcp_frame: type fixed, parent panda_hand, child panda_hand_tcp, origin xyz=2.51535e-17 2.34694e-17 0.16786 rpy=-1.22465e-16 6.12323e-17 -4.59169e-49, axis 0 0 0
- added joint panda_leftfinger_pad_frame: type fixed, parent panda_leftfinger, child panda_leftfinger_pad, origin xyz=0.11668 -0.0134056 -0.009 rpy=3.14159 -1.5708 0, axis 0 0 0
- added joint panda_rightfinger_pad_frame: type fixed, parent panda_rightfinger, child panda_rightfinger_pad, origin xyz=0.11668 0.0134056 -0.009 rpy=-3.14159 -1.5708 0, axis 0 0 0
- joint panda_finger_joint1: axis 0 1 0 -> 0 0 1; limit lower=0.0 upper=0.04 effort=100 velocity=0.2 -> lower=-0.185 upper=0.5 effort=100 velocity=10; mimic (none) -> joint=panda_finger_joint2 multiplier=1.0; origin xyz=0 0 0.0584 rpy=0 0 0 -> xyz=0.00902 -0.0134056 0.0511842 rpy=-1.5708 -1.38679 -1.5708; type prismatic -> revolute
- joint panda_finger_joint2: axis 0 -1 0 -> 0 0 -1; limit lower=0.0 upper=0.04 effort=100 velocity=0.2 -> lower=-0.185 upper=0.5 effort=100 velocity=10; mimic joint=panda_finger_joint1 -> (none); origin xyz=0 0 0.0584 rpy=0 0 0 -> xyz=0.00902 0.0134056 0.0511842 rpy=1.5708 -1.38679 1.5708; type prismatic -> revolute
- joint panda_hand_joint: origin xyz=0 0 0 rpy=0 0 -0.7853981633974483 -> xyz=0 0 0 rpy=0 0 0

Commit message: t

File: mani_skill/assets/robots/panda/panda_v2.urdf (robot description, URDF)
Before this commit: robot panda, 16 links, 15 joints
Links:
- link panda_rightfinger: mass 0.0320815 -> 0.0322882

Commit message: ok

File: mani_skill/assets/robots/panda/panda_v2.urdf (robot description, URDF)
Before this commit: robot panda, 16 links, 15 joints
Joints:
- joint panda_hand_joint: origin xyz=0 0 0 rpy=0 0 0 -> xyz=0 0 0 rpy=0 0 0.698

Commit message: t

File: mani_skill/assets/robots/panda/panda_v2.urdf (robot description, URDF)
Before this commit: robot panda, 16 links, 15 joints
Joints:
- joint panda_hand_joint: origin xyz=0 0 0 rpy=0 0 0.698 -> xyz=0 0 0 rpy=0 0 0.7853981633974483

Commit message: t

File: mani_skill/assets/robots/panda/panda_v2.urdf (robot description, URDF)
Before this commit: robot panda, 16 links, 15 joints
Links:
- removed link panda_hand_1
- link panda_hand: mass 0.0837641 -> 0.73; geometry collision mesh filename=franka_description/meshes/collision/hand.stl; visual mesh filename=franka_description/meshes/visual/hand.glb
- link panda_hand_tcp: mass 1e-9 -> None
- link panda_leftfinger: mass 0.0322882 -> 0.015; geometry collision box size=17.5e-3 15.2e-3 18.5e-3; collision box size=17.5e-3 7e-3 23.5e-3
- link panda_leftfinger_pad: mass 1e-9 -> None
- link panda_rightfinger: mass 0.0322882 -> 0.015; geometry collision box size=17.5e-3 15.2e-3 18.5e-3; collision box size=17.5e-3 7e-3 23.5e-3
- link panda_rightfinger_pad: mass 1e-9 -> None
Joints:
- removed joint panda_hand_1_frame
- removed joint panda_hand_tcp_frame
- removed joint panda_leftfinger_pad_frame
- removed joint panda_rightfinger_pad_frame
- added joint panda_hand_tcp_joint: type fixed, parent panda_hand, child panda_hand_tcp, origin xyz=0 0 0.1034 rpy=0 0 0
- added joint panda_leftfinger_pad_joint: type fixed, parent panda_leftfinger, child panda_leftfinger_pad, origin xyz=0 0 0.0455 rpy=0 0 0
- added joint panda_rightfinger_pad_joint: type fixed, parent panda_rightfinger, child panda_rightfinger_pad, origin xyz=0 0 0.0455 rpy=0 0 0
- joint panda_finger_joint1: axis 0 0 1 -> 0 1 0; limit lower=-0.185 upper=0.5 effort=100 velocity=10 -> lower=0.0 upper=0.04 effort=100 velocity=0.2; mimic joint=panda_finger_joint2 multiplier=1.0 -> (none); origin xyz=0.00902 -0.0134056 0.0511842 rpy=-1.5708 -1.38679 -1.5708 -> xyz=0 0 0.0584 rpy=0 0 0; type revolute -> prismatic
- joint panda_finger_joint2: axis 0 0 -1 -> 0 -1 0; limit lower=-0.185 upper=0.5 effort=100 velocity=10 -> lower=0.0 upper=0.04 effort=100 velocity=0.2; mimic (none) -> joint=panda_finger_joint1; origin xyz=0.00902 0.0134056 0.0511842 rpy=1.5708 -1.38679 1.5708 -> xyz=0 0 0.0584 rpy=0 0 0; type revolute -> prismatic
- joint panda_hand_joint: origin xyz=0 0 0 rpy=0 0 0.7853981633974483 -> xyz=0 0 0 rpy=0 0 -0.7853981633974483

Commit message: t

File: mani_skill/assets/robots/panda/panda_v2.urdf (robot description, URDF)
Before this commit: robot panda, 15 links, 14 joints
Links:
- added link panda_hand_1, mass 1e-9
- link panda_hand: mass 0.73 -> 0.01; geometry collision mesh filename=gripper/convex_decomposition/part_3_parts_00000.stl; collision mesh filename=gripper/convex_decomposition/part_3_parts_00001.stl
- link panda_hand_tcp: mass None -> 1e-9
- link panda_leftfinger: mass 0.015 -> 0.0322882; geometry collision mesh filename=gripper/convex_decomposition/panda_leftfinger_parts_00000.s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; collision mesh filename=gripper/convex_decomposition/panda_leftfinger_parts_00001.s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
- link panda_leftfinger_pad: mass None -> 1e-9
- link panda_rightfinger: mass 0.015 -> 0.0322882; geometry collision mesh filename=gripper/convex_decomposition/panda_rightfinger_parts_00000.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; collision mesh filename=gripper/convex_decomposition/panda_rightfinger_parts_00001.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
- link panda_rightfinger_pad: mass None -> 1e-9
Joints:
- removed joint panda_hand_tcp_joint
- removed joint panda_leftfinger_pad_joint
- removed joint panda_rightfinger_pad_joint
- added joint panda_hand_1_frame: type fixed, parent panda_hand, child panda_hand_1, origin xyz=1.47451e-17 2.91244e-18 0 rpy=-1.22465e-16 6.12323e-17 -4.59169e-49, axis 0 0 0
- added joint panda_hand_tcp_frame: type fixed, parent panda_hand, child panda_hand_tcp, origin xyz=2.51535e-17 2.34694e-17 0.16786 rpy=-1.22465e-16 6.12323e-17 -4.59169e-49, axis 0 0 0
- added joint panda_leftfinger_pad_frame: type fixed, parent panda_leftfinger, child panda_leftfinger_pad, origin xyz=0.11668 -0.0134056 -0.009 rpy=3.14159 -1.5708 0, axis 0 0 0
- added joint panda_rightfinger_pad_frame: type fixed, parent panda_rightfinger, child panda_rightfinger_pad, origin xyz=0.11668 0.0134056 -0.009 rpy=-3.14159 -1.5708 0, axis 0 0 0
- joint panda_finger_joint1: axis 0 1 0 -> 0 0 1; limit lower=0.0 upper=0.04 effort=100 velocity=0.2 -> lower=-0.185 upper=0.5 effort=100 velocity=10; mimic (none) -> joint=panda_finger_joint2 multiplier=1.0; origin xyz=0 0 0.0584 rpy=0 0 0 -> xyz=0.00902 -0.0134056 0.0511842 rpy=-1.5708 -1.38679 -1.5708; type prismatic -> revolute
- joint panda_finger_joint2: axis 0 -1 0 -> 0 0 -1; limit lower=0.0 upper=0.04 effort=100 velocity=0.2 -> lower=-0.185 upper=0.5 effort=100 velocity=10; mimic joint=panda_finger_joint1 -> (none); origin xyz=0 0 0.0584 rpy=0 0 0 -> xyz=0.00902 0.0134056 0.0511842 rpy=1.5708 -1.38679 1.5708; type prismatic -> revolute

Commit message: t

File: mani_skill/assets/robots/panda/panda_v2.urdf (robot description, URDF)
Before this commit: robot panda, 16 links, 15 joints
Links:
- link panda_hand: mass 0.01 -> 0.0837641

Commit message: t

File: mani_skill/assets/robots/panda/panda_v2.urdf (robot description, URDF)
Before this commit: robot panda, 16 links, 15 joints
Links:
- removed link panda_hand_1
- link panda_hand: mass 0.0837641 -> 0.0835752; geometry collision mesh filename=gripper/convex_decomposition/panda_hand_parts_00000.stl; collision mesh filename=gripper/convex_decomposition/panda_hand_parts_00001.stl
- link panda_leftfinger: mass 0.0322882 -> 0.0318189
- link panda_rightfinger: mass 0.0322882 -> 0.031612
Joints:
- removed joint panda_hand_1_frame
- joint panda_finger_joint1: limit lower=-0.185 upper=0.5 effort=100 velocity=10 -> lower=0 upper=0.69 effort=10 velocity=10; origin xyz=0.00902 -0.0134056 0.0511842 rpy=-1.5708 -1.38679 -1.5708 -> xyz=0.00902 -0.0134056 0.0511842 rpy=-3.14159 -1.5708 0
- joint panda_finger_joint2: axis 0 0 -1 -> 0 0 1; limit lower=-0.185 upper=0.5 effort=100 velocity=10 -> lower=0 upper=0.69 effort=10 velocity=10; origin xyz=0.00902 0.0134056 0.0511842 rpy=1.5708 -1.38679 1.5708 -> xyz=0.00902 0.0134056 0.0511842 rpy=3.14159 -1.5708 0
- joint panda_hand_tcp_frame: origin xyz=2.51535e-17 2.34694e-17 0.16786 rpy=-1.22465e-16 6.12323e-17 -4.59169e-49 -> xyz=2.42861e-17 2.19998e-17 0.15586 rpy=-1.22465e-16 6.12323e-17 -4.59169e-49
- joint panda_leftfinger_pad_frame: origin xyz=0.11668 -0.0134056 -0.009 rpy=3.14159 -1.5708 0 -> xyz=0.10468 -0.0134056 -0.009 rpy=3.14159 -1.5708 0
- joint panda_rightfinger_pad_frame: origin xyz=0.11668 0.0134056 -0.009 rpy=-3.14159 -1.5708 0 -> xyz=0.10468 0.0134056 -0.009 rpy=-3.14159 -1.5708 0

File: mani_skill/assets/robots/panda/panda_v2_3.urdf (robot description, URDF)
Before this commit: robot panda, 16 links, 15 joints
Links:
- removed link part_3
- added link panda_hand_1, mass 1e-9
- link panda_hand: mass 1e-9 -> 0.0837641; geometry collision mesh filename=gripper/convex_decomposition/part_3_parts_00000.stl; collision mesh filename=gripper/convex_decomposition/part_3_parts_00001.stl
- link panda_rightfinger: mass 0.0320815 -> 0.0322882
Joints:
- removed joint panda_hand_frame
- added joint panda_hand_1_frame: type fixed, parent panda_hand, child panda_hand_1, origin xyz=1.47451e-17 2.91244e-18 0 rpy=-1.22465e-16 6.12323e-17 -4.59169e-49, axis 0 0 0
- joint panda_finger_joint1: limit lower=0 upper=0.69 effort=10 velocity=0.3 -> lower=-0.185 upper=0.5 effort=100 velocity=10; origin xyz=-0.10918 0.0134056 0.015 rpy=0 0 0 -> xyz=0.00902 -0.0134056 0.0511842 rpy=-1.5708 -1.38679 -1.5708; parent part_3 -> panda_hand
- joint panda_finger_joint2: limit lower=0 upper=0.69 effort=10 velocity=0.3 -> lower=-0.185 upper=0.5 effort=100 velocity=10; origin xyz=-0.10918 -0.0134056 0.015 rpy=0 0 0 -> xyz=0.00902 0.0134056 0.0511842 rpy=1.5708 -1.38679 1.5708; parent part_3 -> panda_hand
- joint panda_hand_joint: child part_3 -> panda_hand; origin xyz=0 0 0.162 rpy=0 -1.5708 2.38562 -> xyz=0 0 0 rpy=0 0 -0.7853981633974483
- joint panda_hand_tcp_frame: origin xyz=0.0074957 -1.73472e-18 0.00598 rpy=0 -6.12323e-17 0 -> xyz=2.51535e-17 2.34694e-17 0.16786 rpy=-1.22465e-16 6.12323e-17 -4.59169e-49; parent part_3 -> panda_hand
- joint panda_leftfinger_pad_frame: origin xyz=0.11668 -0.0134056 -0.009 rpy=6.12323e-17 7.88861e-31 -3.46945e-16 -> xyz=0.11668 -0.0134056 -0.009 rpy=3.14159 -1.5708 0
- joint panda_rightfinger_pad_frame: origin xyz=0.11668 0.0134056 -0.009 rpy=-6.12323e-17 -2.80596e-32 3.46945e-16 -> xyz=0.11668 0.0134056 -0.009 rpy=-3.14159 -1.5708 0

Commit message: t

File: mani_skill/assets/robots/panda/panda_v2.urdf (robot description, URDF)
Before this commit: robot panda, 15 links, 14 joints
Joints:
- joint panda_finger_joint2: axis 0 0 1 -> 0 0 -1

Commit message: t

File: mani_skill/assets/robots/panda/panda_v2.urdf (robot description, URDF)
Before this commit: robot panda, 15 links, 14 joints
Links:
- link panda_hand: geometry collision mesh filename=gripper/convex_decomposition/panda_hand_parts_00000.stl; collision mesh filename=gripper/convex_decomposition/panda_hand_parts_00001.stl

Commit message: 不要凸包

File: mani_skill/assets/robots/panda/panda_v2.urdf (robot description, URDF)
Before this commit: robot panda, 15 links, 14 joints
Links:
- link panda_hand: geometry collision mesh filename=gripper/merged/panda_hand_collision.stl; visual mesh filename=gripper/merged/panda_hand_visual.stl
- link panda_leftfinger: geometry collision mesh filename=gripper/merged/panda_leftfinger_collision.stl; visual mesh filename=gripper/merged/panda_leftfinger_visual.stl
- link panda_rightfinger: geometry collision mesh filename=gripper/merged/panda_rightfinger_collision.stl; visual mesh filename=gripper/merged/panda_rightfinger_visual.stl

Commit message: Revert "不要凸包"
This reverts commit d1fbad073f4b372777d5bf11711fe6e962f63243.

File: mani_skill/assets/robots/panda/panda_v2.urdf (robot description, URDF)
Before this commit: robot panda, 15 links, 14 joints
Links:
- link panda_hand: geometry collision mesh filename=gripper/convex_decomposition/panda_hand_parts_00000.stl; collision mesh filename=gripper/convex_decomposition/panda_hand_parts_00001.stl
- link panda_leftfinger: geometry collision mesh filename=gripper/convex_decomposition/panda_leftfinger_parts_00000.s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; collision mesh filename=gripper/convex_decomposition/panda_leftfinger_parts_00001.s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
- link panda_rightfinger: geometry collision mesh filename=gripper/convex_decomposition/panda_rightfinger_parts_00000.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; collision mesh filename=gripper/convex_decomposition/panda_rightfinger_parts_00001.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

Commit message: 测试

File: mani_skill/assets/robots/panda/panda_v2.urdf (robot description, URDF)
Before this commit: robot panda, 15 links, 14 joints
Links:
- added link camera_link, mass 1e-9
Joints:
- added joint camera_link_frame: type fixed, parent panda_hand, child camera_link, origin xyz=0.07382 -0.00025 0.0305842 rpy=-6.12323e-17 -1.14553e-15 -2.00965e-31, axis 0 0 0

Commit message: ok

File: mani_skill/assets/robots/panda/panda_v2.urdf (robot description, URDF)
Before this commit: robot panda, 16 links, 15 joints
Joints:
- joint camera_link_frame: origin xyz=0.07382 -0.00025 0.0305842 rpy=-6.12323e-17 -1.14553e-15 -2.00965e-31 -> xyz=0.07382 -0.00025 0.0405842 rpy=-6.12323e-17 -1.14553e-15 -2.00965e-31

Commit message: ok

File: mani_skill/assets/robots/panda/panda_v2.urdf (robot description, URDF)
Before this commit: robot panda, 16 links, 15 joints
Joints:
- joint camera_link_frame: origin xyz=0.07382 -0.00025 0.0405842 rpy=-6.12323e-17 -1.14553e-15 -2.00965e-31 -> xyz=0.07382 -0.00025 0.0395842 rpy=-6.12323e-17 -1.14553e-15 -2.00965e-31
